Commit message: Initial commit

File: cpr_inspection_gazebo/urdf/inspection_geometry.urdf.xacro (robot description, xacro)
@@ -10,5 +10,5 @@
       <origin xyz="0 0 0" rpy="0 0 0"/>
       <geometry>
-        <mesh filename="package://cpr_inspection_gazebo/meshes/inspection_world.dae"/>
+        <mesh filename="package://cpr_inspection_gazebo/meshes/inspection_world_copy.dae"/>
       </geometry>
     </visual>
@@ -16,5 +16,5 @@
       <origin xyz="0 0 0" rpy="0 0 0"/>
       <geometry>
-        <mesh filename="package://cpr_inspection_gazebo/meshes/inspection_world.dae"/>
+        <mesh filename="package://cpr_inspection_gazebo/meshes/inspection_world_copy.dae"/>
       </geometry>
       <surface>
